Commit message: 准备移植宇树官方开源slam算法到ros2上

File: install/go2_description/share/go2_description/urdf/go2_description.urdf (robot description, URDF)
Before this commit: robot go2_description, 29 links, 28 joints
Links:
- removed link radar
- added link utlidar_lidar, mass 0
Joints:
- joint radar_joint: child radar -> utlidar_lidar

Commit message: 更换为师兄训练策略，测试基本通过，可能存在扰动鲁棒性问题，待询问

File: install/go2_description/share/go2_description/urdf/go2_description.urdf (robot description, URDF)
Before this commit: robot go2_description, 29 links, 28 joints
Links:
- added link back_payload, mass 1.0; collision box size=0.2 0.15 0.1; visual box size=0.2 0.15 0.1
Joints:
- added joint back_payload_joint: type fixed, parent base, child back_payload, origin xyz=-0.03 0 0.132 rpy=0 0 0

Commit message: 添加eth高程图包，基本测试通过

File: install/go2_description/share/go2_description/urdf/go2_description.urdf (robot description, URDF)
Before this commit: robot go2_description, 30 links, 29 joints
Links:
- added link lidar_mid360, mass 0.265; collision box size=0.065 0.065 0.06; visual box size=0.065 0.065 0.06
Joints:
- added joint lidar_mid360_joint: type fixed, parent base, child lidar_mid360, origin xyz=0.31 0 0.18 rpy=0 0.7853981634 0
